Commit message: Updated

File: kuka_description/urdf/dim_kuka.xacro (robot description, xacro)
@@ -1,5 +1,5 @@
 <?xml version="1.0" ?>
 <robot name="kuka_kr4r600" xmlns:xacro="http://wiki.ros.org/xacro">
-  <xacro:include filename="$(find kuka_description)/urdf/kr4r600_macro.xacro"/>
+  <xacro:include filename="$(find kuka_description)/urdf/dim_kuka_macro.xacro"/>
   <xacro:kuka_kr4r600 prefix=""/>
 </robot>

File: kuka_description/urdf/kr4r600_macro.xacro (robot description, xacro)
@@ -17,5 +17,5 @@
   <!-- <xacro:macro name="kuka_kr4r600" params="prefix"> -->
     <link name="${prefix}base_link">
-    <xacro:default_inertial mass="1"/>
+    <xacro:default_inertial mass="100"/>
       <visual>
         <origin xyz="0 0 0" rpy="0 0 0" />
@@ -284,4 +284,87 @@
       <child link="hokuyo_link"/>
     </joint>
+    <transmission name="link_1_trans">
+	<type>transmission_interface/SimpleTransmission</type>
+	<joint name="joint_a1">
+	<hardwareInterface>hardware_interface/PositionJointInterface</hardwareInterface>
+	</joint>
+	<actuator name="link_1_motor">
+	<hardwareInterface>hardware_interface/PositionJointInterface</hardwareInterface>
+	<mechanicalReduction>1</mechanicalReduction>
+	</actuator>
+    </transmission>
+    <transmission name="link_2_trans">
+	<type>transmission_interface/SimpleTransmission</type>
+	<joint name="joint_a2">
+	<hardwareInterface>hardware_interface/PositionJointInterface</hardwareInterface>
+	</joint>
+	<actuator name="link_2_motor">
+	<hardwareInterface>hardware_interface/PositionJointInterface</hardwareInterface>
+	<mechanicalReduction>1</mechanicalReduction>
+	</actuator>
+    </transmission>
+    <transmission name="link_3_trans">
+	<type>transmission_interface/SimpleTransmission</type>
+	<joint name="joint_a3">
+	<hardwareInterface>hardware_interface/PositionJointInterface</hardwareInterface>
+	</joint>
+	<actuator name="link_3_motor">
+	<hardwareInterface>hardware_interface/PositionJointInterface</hardwareInterface>
+	<mechanicalReduction>1</mechanicalReduction>
+	</actuator>
+    </transmission>
+    <transmission name="link_4_trans">
+	<type>transmission_interface/SimpleTransmission</type>
+	<joint name="joint_a4">
+	<hardwareInterface>hardware_interface/PositionJointInterface</hardwareInterface>
+	</joint>
+	<actuator name="link_4_motor">
+	<hardwareInterface>hardware_interface/PositionJointInterface</hardwareInterface>
+	<mechanicalReduction>1</mechanicalReduction>
+	</actuator>
+    </transmission>
+    <transmission name="link_5_trans">
+	<type>transmission_interface/SimpleTransmission</type>
+	<joint name="joint_a5">
+	<hardwareInterface>hardware_interface/PositionJointInterface</hardwareInterface>
+	</joint>
+	<actuator name="link_5_motor">
+	<hardwareInterface>hardware_interface/PositionJointInterface</hardwareInterface>
+	<mechanicalReduction>1</mechanicalReduction>
+	</actuator>
+    </transmission>
+    <transmission name="link_6_trans">
+	<type>transmission_interface/SimpleTransmission</type>
+	<joint name="joint_a6">
+	<hardwareInterface>hardware_interface/PositionJointInterface</hardwareInterface>
+	</joint>
+	<actuator name="link_6_motor">
+	<hardwareInterface>hardware_interface/PositionJointInterface</hardwareInterface>
+	<mechanicalReduction>1</mechanicalReduction>
+	</actuator>
+    </transmission>
+    <gazebo>
+	<plugin name="control" filename="libgazebo_ros_control.so">
+	<robotNamespace>/</robotNamespace>
+	</plugin>
+    </gazebo>
+    <gazebo reference="link_1">
+	<selfCollide>true</selfCollide>
+    </gazebo>
+    <gazebo reference="link_2">
+	<selfCollide>true</selfCollide>
+    </gazebo>
+    <gazebo reference="link_3">
+	<selfCollide>true</selfCollide>
+    </gazebo>
+    <gazebo reference="link_4">
+	<selfCollide>true</selfCollide>
+    </gazebo>
+    <gazebo reference="link_5">
+	<selfCollide>true</selfCollide>
+    </gazebo>
+    <gazebo reference="link_6">
+	<selfCollide>true</selfCollide>
+    </gazebo>
 <!--   <xacro:kuka_arm_transmission prefix="${prefix}" hw_interface="${transmission_hw_interface}" />
   <xacro:kuka_arm_gazebo prefix="${prefix}" />

File: kuka_description/urdf/kuka_kr4r600_macro.xacro (robot description, xacro)
@@ -60,6 +60,29 @@
   </transmission>
   <!-- end of transmission list -->
+     <gazebo>
+	<plugin name="control" filename="libgazebo_ros_control.so">
+	<robotNamespace>/</robotNamespace>
+	</plugin>
+    </gazebo>
+    <gazebo reference="link_1">
+	<selfCollide>true</selfCollide>
+    </gazebo>
+    <gazebo reference="link_2">
+	<selfCollide>true</selfCollide>
+    </gazebo>
+    <gazebo reference="link_3">
+	<selfCollide>true</selfCollide>
+    </gazebo>
+    <gazebo reference="link_4">
+	<selfCollide>true</selfCollide>
+    </gazebo>
+    <gazebo reference="link_5">
+	<selfCollide>true</selfCollide>
+    </gazebo>
+    <gazebo reference="link_6">
+	<selfCollide>true</selfCollide>
+    </gazebo>
   <!-- Gazebo-specific link properties -->
-  <gazebo reference="${prefix}base_link">
+  <!--gazebo reference="${prefix}base_link">
     <material>Gazebo/White</material>
     <turnGravityOff>true</turnGravityOff>
@@ -88,5 +111,5 @@
     <material>Gazebo/Black</material>
     <turnGravityOff>true</turnGravityOff>
-  </gazebo>
+  </gazebo-->
   <!-- ros_control plugin -->
   <gazebo>

File: kuka_description/urdf/table.urdf.xacro (robot description, xacro)
@@ -24,4 +24,5 @@
   <xacro:property name="table_top_thickness" value="0.05"/>
   <xacro:property name="M_PI" value="3.1415926535897931" />
+  <xacro:include filename="$(find kuka_description)/urdf/container.xacro"/>
   <!-- tabletop height is .55+.01+.025=.585 -->
   <link name="table_top_link">
